Commit message: [ADD] add camera depth optical joint and frame

File: orbbec_description/urdf/gemini_335_L_336_L_macro.urdf.xacro (robot description, xacro)
@@ -70,4 +70,11 @@
       <axis xyz="0 0 0" />
     </joint>
+    <joint name="${tf_prefix}camera_depth_optical_joint" type="fixed">
+      <origin xyz="0 0 0" rpy="-1.5708 0 -1.5708" />
+      <parent link="${tf_prefix}camera_depth_frame" />
+      <child link="${tf_prefix}camera_depth_optical_frame" />
+      <axis xyz="0 0 0" />
+    </joint>
+    <link name="${tf_prefix}camera_depth_optical_frame" />
     <link name="${tf_prefix}camera_IMU_frame">
       <inertial>
